File: Pico Robotic Controller.kicad_pcb (KiCad board)
At the start: 4 copper layers, 91 x 110 mm, 100 parts, among them J1 250-202, J10 Conn_02x03_Odd_Even, J11 250-202, J12 250-202, J13 Conn_02x05_Odd_Even, J2 conn_04_03, J3 250-203, J4 conn_04_03, J5 Conn_01x03, J6 Conn_01x02, J7 conn_04_03, J8 conn_04_03, J9 Conn_01x03, Q1 DMG2305UX-13, U1 Weewooday-820, U10 APX321WG-7, U11 74HC14, U12 74HC14, U13 PCA9685PW, U2 RPi_Pico_W, U3 RPi_Picobell_CAN_Bus, U4 PCA9685PW, U5 TCA9546, U6 Ethernet_FeatherWing, U7 TXS0104EPW, U8 TXS0104EPW, U9 APX321WG-7, X1 STEMMA_I2C_QT, X2 STEMMA_I2C_QT, X3 STEMMA_I2C_QT, X4 STEMMA_I2C_QT

Commit message: updated design files that correct a silkscreen comment (2023 to 2024)
Other:
- board text added: "PCB Made in 2024"
- board text removed: "PCB Made in 2023"

Commit message: updated KiCAD design files to add separate OEn for motor PWM generator
Parts:
- added G***: LOGO, LOGO, B.Cu at (140.5, 99.7)
- added G***: LOGO, LOGO, B.Cu at (138.6, 126.7)
- added R18: 5K1, Resistor_SMD:R_1206_3216Metric, F.Cu at (162.2, 137.2)
- R10, R11, R12, R13, R14, R15, R16, R17: value R_Small -> 13
- moved R3 14.8 mm to (160.4, 122.5)
Connections:
- R3 pad 2: /PWM_OEn -> /MOTOR_OEn
- U13 pad 23: /PWM_OEn -> /MOTOR_OEn
- U2 pad 34: unconnected-(U2-Pad34) -> /MOTOR_OEn
Routing:
- net /MOTOR_OEn: track 0.00 -> 42.0 mm
- net /PWM_OEn: track 39.7 -> 21.4 mm
- net GND: track 137.7 -> 138.9 mm, vias 74 -> 75
Other:
- board text added: "Designed by Scott McMahon Mentor of FRC2468, 2687, and 2689 A low-cost prototyping platform that has similarities to the XRP platform (Pico W based) plus the interfacing of the roboRIO. Intended to reduce prototyping cost by providing a cheaper platform plus de-risk using a roboRIO."

Commit message: updated the PWM generator enables to be pull ups from pull down
Connections:
- R18 pad 1: GND -> +3V3
- R3 pad 1: GND -> +3V3
Routing:
- net GND: track 138.9 -> 135.9 mm, vias 75 -> 74
